Commit message: made two files to find inertia issues

File: urdf/ability_hand_right_gazebo.urdf (robot description, URDF)
Before this commit: robot ability_hand, 17 links, 16 joints
Links:
- added link world
- link base: geometry collision mesh filename=package://ability_hand_sim/meshes/wristmesh.STL; visual mesh filename=package://ability_hand_sim/meshes/wristmesh.STL
- link index_L1: geometry collision mesh filename=package://ability_hand_sim/meshes/idx-F1.STL; visual mesh filename=package://ability_hand_sim/meshes/idx-F1.STL
- link index_L2: geometry collision mesh filename=package://ability_hand_sim/meshes/idx-F2.STL; visual mesh filename=package://ability_hand_sim/meshes/idx-F2.STL
- link middle_L1: geometry collision mesh filename=package://ability_hand_sim/meshes/idx-F1.STL; visual mesh filename=package://ability_hand_sim/meshes/idx-F1.STL
- link middle_L2: geometry collision mesh filename=package://ability_hand_sim/meshes/idx-F2.STL; visual mesh filename=package://ability_hand_sim/meshes/idx-F2.STL
- link pinky_L1: geometry collision mesh filename=package://ability_hand_sim/meshes/idx-F1.STL; visual mesh filename=package://ability_hand_sim/meshes/idx-F1.STL
- link pinky_L2: geometry collision mesh filename=package://ability_hand_sim/meshes/idx-F2.STL; visual mesh filename=package://ability_hand_sim/meshes/idx-F2.STL
- link ring_L1: geometry collision mesh filename=package://ability_hand_sim/meshes/idx-F1.STL; visual mesh filename=package://ability_hand_sim/meshes/idx-F1.STL
- link ring_L2: geometry collision mesh filename=package://ability_hand_sim/meshes/idx-F2.STL; visual mesh filename=package://ability_hand_sim/meshes/idx-F2.STL
- link thumb_L1: geometry collision mesh filename=package://ability_hand_sim/meshes/thumb-F1-MIR.STL; visual mesh filename=package://ability_hand_sim/meshes/thumb-F1-MIR.STL
- link thumb_L2: geometry collision mesh filename=package://ability_hand_sim/meshes/thumb-F2.STL; visual mesh filename=package://ability_hand_sim/meshes/thumb-F2.STL
- link thumb_base: geometry collision mesh filename=package://ability_hand_sim/meshes/FB_palm_ref_MIR.STL; visual mesh filename=package://ability_hand_sim/meshes/FB_palm_ref_MIR.STL
Joints:
- added joint grounding : type fixed, parent world, child base, origin xyz=0. 0. 0. rpy=0. 0. 0.
